Commit message: Update humanoid URDF description and mesh files

File: URDF_F_description/URDF_F_description/urdf/URDF_F.xacro (robot description, xacro)
@@ -6,7 +6,7 @@
 <link name="base_link">
   <inertial>
-    <origin xyz="2.6645352591003753e-17 1.1102230246251557e-17 0.4919999999999998" rpy="0 0 0"/>
+    <origin xyz="-0.009999999999993764 0.0029999999999999498 0.491999999999998" rpy="0 0 0"/>
     <mass value="1.9999999999999996"/>
-    <inertia ixx="0.002083" iyy="0.007083" izz="0.008333" ixy="0.0" iyz="-0.0" ixz="0.0"/>
+    <inertia ixx="0.002083" iyy="0.007083" izz="0.008333" ixy="0.0" iyz="0.0" ixz="0.0"/>
   </inertial>
   <visual>
@@ -24,172 +24,12 @@
   </collision>
 </link>
-<link name="foot_L_1">
-  <inertial>
-    <origin xyz="-2.7755575615628914e-17 9.755025872021025e-05 -0.02861035771693201" rpy="0 0 0"/>
-    <mass value="0.3"/>
-    <inertia ixx="0.000345" iyy="0.000167" izz="0.000392" ixy="-0.0" iyz="1e-05" ixz="-0.0"/>
-  </inertial>
-  <visual>
-    <origin xyz="-0.077 0.0245 -0.04" rpy="0 0 0"/>
-    <geometry>
-      <mesh filename="file://$(find URDF_F_description)/meshes/foot_L_1.stl" scale="0.001 0.001 0.001"/>
-    </geometry>
-    <material name="silver"/>
-  </visual>
-  <collision>
-    <origin xyz="-0.077 0.0245 -0.04" rpy="0 0 0"/>
-    <geometry>
-      <mesh filename="file://$(find URDF_F_description)/meshes/foot_L_1.stl" scale="0.001 0.001 0.001"/>
-    </geometry>
-  </collision>
-</link>
-<link name="footJ_L_1">
-  <inertial>
-    <origin xyz="-0.02132600000000008 0.014075999999998895 -0.04228105550025508" rpy="0 0 0"/>
-    <mass value="0.06"/>
-    <inertia ixx="3.2e-05" iyy="4.3e-05" izz="3e-05" ixy="0.0" iyz="-0.0" ixz="-0.0"/>
-  </inertial>
-  <visual>
-    <origin xyz="-0.098326 0.017076 -0.08" rpy="0 0 0"/>
-    <geometry>
-      <mesh filename="file://$(find URDF_F_description)/meshes/footJ_L_1.stl" scale="0.001 0.001 0.001"/>
-    </geometry>
-    <material name="silver"/>
-  </visual>
-  <collision>
-    <origin xyz="-0.098326 0.017076 -0.08" rpy="0 0 0"/>
-    <geometry>
-      <mesh filename="file://$(find URDF_F_description)/meshes/footJ_L_1.stl" scale="0.001 0.001 0.001"/>
-    </geometry>
-  </collision>
-</link>
-<link name="AK45-10_frL_1">
-  <inertial>
-    <origin xyz="-0.077 0.044499999999999 0.024999784125248788" rpy="0 0 0"/>
-    <mass value="0.26"/>
-    <inertia ixx="7.7e-05" iyy="7.4e-05" izz="7.7e-05" ixy="0.0" iyz="-0.0" ixz="0.0"/>
-  </inertial>
-  <visual>
-    <origin xyz="-0.154 0.0475 -0.015" rpy="0 0 0"/>
-    <geometry>
-      <mesh filename="file://$(find URDF_F_description)/meshes/AK45-10_frL_1.stl" scale="0.001 0.001 0.001"/>
-    </geometry>
-    <material name="silver"/>
-  </visual>
-  <collision>
-    <origin xyz="-0.154 0.0475 -0.015" rpy="0 0 0"/>
-    <geometry>
-      <mesh filename="file://$(find URDF_F_description)/meshes/AK45-10_frL_1.stl" scale="0.001 0.001 0.001"/>
-    </geometry>
-  </collision>
-</link>
-<link name="calf_L_1">
-  <inertial>
-    <origin xyz="-0.0018470097394905627 -1.8214596497756474e-17 -0.08050979935301733" rpy="0 0 0"/>
-    <mass value="0.5"/>
-    <inertia ixx="0.001191" iyy="0.001287" izz="0.0002104" ixy="0.0" iyz="-0.0" ixz="7.1e-05"/>
-  </inertial>
-  <visual>
-    <origin xyz="-0.077 0.003 -0.24" rpy="0 0 0"/>
-    <geometry>
-      <mesh filename="file://$(find URDF_F_description)/meshes/calf_L_1.stl" scale="0.001 0.001 0.001"/>
-    </geometry>
-    <material name="silver"/>
-  </visual>
-  <collision>
-    <origin xyz="-0.077 0.003 -0.24" rpy="0 0 0"/>
-    <geometry>
-      <mesh filename="file://$(find URDF_F_description)/meshes/calf_L_1.stl" scale="0.001 0.001 0.001"/>
-    </geometry>
-  </collision>
-</link>
-<link name="AK45-36_tpL_1">
-  <inertial>
-    <origin xyz="-0.04999999999999999 0.0030000000000000053 -0.37000000000000144" rpy="0 0 0"/>
-    <mass value="0.34"/>
-    <inertia ixx="0.000099" iyy="0.000132" izz="0.000132" ixy="0.0" iyz="0.0" ixz="-0.0"/>
-  </inertial>
-  <visual>
-    <origin xyz="-0.1 0.006 -0.74" rpy="0 0 0"/>
-    <geometry>
-      <mesh filename="file://$(find URDF_F_description)/meshes/AK45-36_tpL_1.stl" scale="0.001 0.001 0.001"/>
-    </geometry>
-    <material name="silver"/>
-  </visual>
-  <collision>
-    <origin xyz="-0.1 0.006 -0.74" rpy="0 0 0"/>
-    <geometry>
-      <mesh filename="file://$(find URDF_F_description)/meshes/AK45-36_tpL_1.stl" scale="0.001 0.001 0.001"/>
-    </geometry>
-  </collision>
-</link>
-<link name="thigh_L_1">
-  <inertial>
-    <origin xyz="-0.00539746230815126 0.0003817221478294966 -0.059989569173888924" rpy="0 0 0"/>
-    <mass value="0.5"/>
-    <inertia ixx="0.000862" iyy="0.001054" izz="0.000388" ixy="3.9e-06" iyz="-6.8e-06" ixz="-6.4e-05"/>
-  </inertial>
-  <visual>
-    <origin xyz="-0.077 0.003 -0.37" rpy="0 0 0"/>
-    <geometry>
-      <mesh filename="file://$(find URDF_F_description)/meshes/thigh_L_1.stl" scale="0.001 0.001 0.001"/>
-    </geometry>
-    <material name="silver"/>
-  </visual>
-  <collision>
-    <origin xyz="-0.077 0.003 -0.37" rpy="0 0 0"/>
-    <geometry>
-      <mesh filename="file://$(find URDF_F_description)/meshes/thigh_L_1.stl" scale="0.001 0.001 0.001"/>
-    </geometry>
-  </collision>
-</link>
-<link name="thighJ_L_1">
-  <inertial>
-    <origin xyz="-0.05000000000000002 0.40677616547554 -0.07845450823157368" rpy="0 0 0"/>
-    <mass value="0.06"/>
-    <inertia ixx="6.7e-05" iyy="6e-05" izz="3.9e-05" ixy="-0.0" iyz="1.3e-05" ixz="-0.0"/>
-  </inertial>
-  <visual>
-    <origin xyz="-0.1 0.418 -0.462" rpy="0 0 0"/>
-    <geometry>
-      <mesh filename="file://$(find URDF_F_description)/meshes/thighJ_L_1.stl" scale="0.001 0.001 0.001"/>
-    </geometry>
-    <material name="silver"/>
-  </visual>
-  <collision>
-    <origin xyz="-0.1 0.418 -0.462" rpy="0 0 0"/>
-    <geometry>
-      <mesh filename="file://$(find URDF_F_description)/meshes/thighJ_L_1.stl" scale="0.001 0.001 0.001"/>
-    </geometry>
-  </collision>
-</link>
-<link name="AK45-36_trL_1">
-  <inertial>
-    <origin xyz="-0.049999999999999996 0.038999999999999965 -0.4400000000000003" rpy="0 0 0"/>
-    <mass value="0.34"/>
-    <inertia ixx="0.000132" iyy="0.000099" izz="0.000132" ixy="0.0" iyz="-0.0" ixz="0.0"/>
-  </inertial>
-  <visual>
-    <origin xyz="-0.1 0.044 -0.88" rpy="0 0 0"/>
-    <geometry>
-      <mesh filename="file://$(find URDF_F_description)/meshes/AK45-36_trL_1.stl" scale="0.001 0.001 0.001"/>
-    </geometry>
-    <material name="silver"/>
-  </visual>
-  <collision>
-    <origin xyz="-0.1 0.044 -0.88" rpy="0 0 0"/>
-    <geometry>
-      <mesh filename="file://$(find URDF_F_description)/meshes/AK45-36_trL_1.stl" scale="0.001 0.001 0.001"/>
-    </geometry>
-  </collision>
-</link>
 <link name="thighJR_L_1">
   <inertial>
-    <origin xyz="0.05 2.6645352591003756e-17 -0.48573212283403455" rpy="0 0 0"/>
+    <origin xyz="0.06000000000000488 -0.0030000000000000564 -0.4857321228340379" rpy="0 0 0"/>
     <mass value="0.06"/>
     <inertia ixx="2.9e-05" iyy="4.2e-05" izz="3.3e-05" ixy="-0.0" iyz="0.0" ixz="0.0"/>
   </inertial>
   <visual>
-    <origin xyz="-0.0 -0.0 -0.934" rpy="0 0 0"/>
+    <origin xyz="0.02 -0.006 -0.934" rpy="0 0 0"/>
     <geometry>
       <mesh filename="file://$(find URDF_F_description)/meshes/thighJR_L_1.stl" scale="0.001 0.001 0.001"/>
@@ -198,5 +38,5 @@
   </visual>
   <collision>
-    <origin xyz="-0.0 -0.0 -0.934" rpy="0 0 0"/>
+    <origin xyz="0.02 -0.006 -0.934" rpy="0 0 0"/>
     <geometry>
       <mesh filename="file://$(find URDF_F_description)/meshes/thighJR_L_1.stl" scale="0.001 0.001 0.001"/>
@@ -204,61 +44,201 @@
   </collision>
 </link>
-<link name="AK45-36_kL_1">
-  <inertial>
-    <origin xyz="-0.10399999999999986 0.002999999999999984 -0.31000000000000144" rpy="0 0 0"/>
-    <mass value="0.4"/>
-    <inertia ixx="0.000116" iyy="0.000155" izz="0.000155" ixy="0.0" iyz="-0.0" ixz="-0.0"/>
-  </inertial>
-  <visual>
-    <origin xyz="-0.18275 0.006 -0.61" rpy="0 0 0"/>
-    <geometry>
-      <mesh filename="file://$(find URDF_F_description)/meshes/AK45-36_kL_1.stl" scale="0.001 0.001 0.001"/>
-    </geometry>
-    <material name="silver"/>
-  </visual>
-  <collision>
-    <origin xyz="-0.18275 0.006 -0.61" rpy="0 0 0"/>
-    <geometry>
-      <mesh filename="file://$(find URDF_F_description)/meshes/AK45-36_kL_1.stl" scale="0.001 0.001 0.001"/>
-    </geometry>
-  </collision>
-</link>
-<link name="AK45-36_fpL_1">
-  <inertial>
-    <origin xyz="-0.020075999999999997 0.01407599999999995 -0.10000000000000142" rpy="0 0 0"/>
+<link name="AK45-36_trL_1">
+  <inertial>
+    <origin xyz="-0.03999999999999455 0.013999999999999964 -0.4670000000000036" rpy="0 0 0"/>
+    <mass value="0.34"/>
+    <inertia ixx="0.000132" iyy="0.000099" izz="0.000132" ixy="-0.0" iyz="0.0" ixz="0.0"/>
+  </inertial>
+  <visual>
+    <origin xyz="-0.08 0.016 -0.907" rpy="0 0 0"/>
+    <geometry>
+      <mesh filename="file://$(find URDF_F_description)/meshes/AK45-36_trL_1.stl" scale="0.001 0.001 0.001"/>
+    </geometry>
+    <material name="silver"/>
+  </visual>
+  <collision>
+    <origin xyz="-0.08 0.016 -0.907" rpy="0 0 0"/>
+    <geometry>
+      <mesh filename="file://$(find URDF_F_description)/meshes/AK45-36_trL_1.stl" scale="0.001 0.001 0.001"/>
+    </geometry>
+  </collision>
+</link>
+<link name="thigh_L_1">
+  <inertial>
+    <origin xyz="-0.00539746230814965 0.00038172214782945324 -0.059989569173891755" rpy="0 0 0"/>
+    <mass value="0.5"/>
+    <inertia ixx="0.000862" iyy="0.001054" izz="0.000388" ixy="3.9e-06" iyz="-6.7e-06" ixz="-6.4e-05"/>
+  </inertial>
+  <visual>
+    <origin xyz="-0.067 0.0 -0.37" rpy="0 0 0"/>
+    <geometry>
+      <mesh filename="file://$(find URDF_F_description)/meshes/thigh_L_1.stl" scale="0.001 0.001 0.001"/>
+    </geometry>
+    <material name="silver"/>
+  </visual>
+  <collision>
+    <origin xyz="-0.067 0.0 -0.37" rpy="0 0 0"/>
+    <geometry>
+      <mesh filename="file://$(find URDF_F_description)/meshes/thigh_L_1.stl" scale="0.001 0.001 0.001"/>
+    </geometry>
+  </collision>
+</link>
+<link name="AK45-36_kpL_1">
+  <inertial>
+    <origin xyz="-0.09400000000000365 -5.800915303664527e-17 -0.43961500000000436" rpy="0 0 0"/>
     <mass value="0.4"/>
     <inertia ixx="0.000116" iyy="0.000155" izz="0.000155" ixy="-0.0" iyz="0.0" ixz="0.0"/>
   </inertial>
   <visual>
-    <origin xyz="-0.097076 0.017076 -0.28" rpy="0 0 0"/>
-    <geometry>
-      <mesh filename="file://$(find URDF_F_description)/meshes/AK45-36_fpL_1.stl" scale="0.001 0.001 0.001"/>
-    </geometry>
-    <material name="silver"/>
-  </visual>
-  <collision>
-    <origin xyz="-0.097076 0.017076 -0.28" rpy="0 0 0"/>
-    <geometry>
-      <mesh filename="file://$(find URDF_F_description)/meshes/AK45-36_fpL_1.stl" scale="0.001 0.001 0.001"/>
-    </geometry>
-  </collision>
-</link>
-<link name="AK45-36_tpR_1">
-  <inertial>
-    <origin xyz="-0.05000000000000004 0.0029999999999999454 0.3699999999999997" rpy="0 0 0"/>
+    <origin xyz="-0.16275 0.0 -0.739615" rpy="0 0 0"/>
+    <geometry>
+      <mesh filename="file://$(find URDF_F_description)/meshes/AK45-36_kpL_1.stl" scale="0.001 0.001 0.001"/>
+    </geometry>
+    <material name="silver"/>
+  </visual>
+  <collision>
+    <origin xyz="-0.16275 0.0 -0.739615" rpy="0 0 0"/>
+    <geometry>
+      <mesh filename="file://$(find URDF_F_description)/meshes/AK45-36_kpL_1.stl" scale="0.001 0.001 0.001"/>
+    </geometry>
+  </collision>
+</link>
+<link name="calf_L_1">
+  <inertial>
+    <origin xyz="-0.0018470097395003188 -8.38633090922969e-17 -0.08050979935301991" rpy="0 0 0"/>
+    <mass value="0.5"/>
+    <inertia ixx="0.001191" iyy="0.00129" izz="0.000211" ixy="-0.0" iyz="0.0" ixz="7.1e-05"/>
+  </inertial>
+  <visual>
+    <origin xyz="-0.067 0.0 -0.24" rpy="0 0 0"/>
+    <geometry>
+      <mesh filename="file://$(find URDF_F_description)/meshes/calf_L_1.stl" scale="0.001 0.001 0.001"/>
+    </geometry>
+    <material name="silver"/>
+  </visual>
+  <collision>
+    <origin xyz="-0.067 0.0 -0.24" rpy="0 0 0"/>
+    <geometry>
+      <mesh filename="file://$(find URDF_F_description)/meshes/calf_L_1.stl" scale="0.001 0.001 0.001"/>
+    </geometry>
+  </collision>
+</link>
+<link name="footJ_L_1">
+  <inertial>
+    <origin xyz="-1.4627188349436437e-14 -1.072264026970011e-16 -0.0022808396255029964" rpy="0 0 0"/>
+    <mass value="0.06"/>
+    <inertia ixx="3.1e-05" iyy="4.2e-05" izz="3.1e-05" ixy="-0.0" iyz="-0.0" ixz="0.0"/>
+  </inertial>
+  <visual>
+    <origin xyz="-0.067 0.0 -0.04" rpy="0 0 0"/>
+    <geometry>
+      <mesh filename="file://$(find URDF_F_description)/meshes/footJ_L_1.stl" scale="0.001 0.001 0.001"/>
+    </geometry>
+    <material name="silver"/>
+  </visual>
+  <collision>
+    <origin xyz="-0.067 0.0 -0.04" rpy="0 0 0"/>
+    <geometry>
+      <mesh filename="file://$(find URDF_F_description)/meshes/footJ_L_1.stl" scale="0.001 0.001 0.001"/>
+    </geometry>
+  </collision>
+</link>
+<link name="AK45-10_frL_1">
+  <inertial>
+    <origin xyz="-1.457167719820518e-14 -9.643358654519792e-17 7.077671781985373e-16" rpy="0 0 0"/>
+    <mass value="0.24"/>
+    <inertia ixx="7.7e-05" iyy="7.4e-05" izz="7.7e-05" ixy="0.0" iyz="0.0" ixz="-0.0"/>
+  </inertial>
+  <visual>
+    <origin xyz="-0.067 0.0 -0.04" rpy="0 0 0"/>
+    <geometry>
+      <mesh filename="file://$(find URDF_F_description)/meshes/AK45-10_frL_1.stl" scale="0.001 0.001 0.001"/>
+    </geometry>
+    <material name="silver"/>
+  </visual>
+  <collision>
+    <origin xyz="-0.067 0.0 -0.04" rpy="0 0 0"/>
+    <geometry>
+      <mesh filename="file://$(find URDF_F_description)/meshes/AK45-10_frL_1.stl" scale="0.001 0.001 0.001"/>
+    </geometry>
+  </collision>
+</link>
+<link name="foot_L_1">
+  <inertial>
+    <origin xyz="-1.5459855617905305e-14 9.755025872117476e-05 -0.028610141842179894" rpy="0 0 0"/>
+    <mass value="0.3"/>
+    <inertia ixx="0.00035" iyy="0.000168" izz="0.0004" ixy="0.0" iyz="1e-05" ixz="0.0"/>
+  </inertial>
+  <visual>
+    <origin xyz="-0.067 0.0215 -0.04" rpy="0 0 0"/>
+    <geometry>
+      <mesh filename="file://$(find URDF_F_description)/meshes/foot_L_1.stl" scale="0.001 0.001 0.001"/>
+    </geometry>
+    <material name="silver"/>
+  </visual>
+  <collision>
+    <origin xyz="-0.067 0.0215 -0.04" rpy="0 0 0"/>
+    <geometry>
+      <mesh filename="file://$(find URDF_F_description)/meshes/foot_L_1.stl" scale="0.001 0.001 0.001"/>
+    </geometry>
+  </collision>
+</link>
+<link name="thighJ_L_1">
+  <inertial>
+    <origin xyz="3.677613769070831e-15 0.020776165475540002 -0.056454508231575606" rpy="0 0 0"/>
+    <mass value="0.06"/>
+    <inertia ixx="6.7e-05" iyy="6e-05" izz="3.9e-05" ixy="0.0" iyz="1.3e-05" ixz="-0.0"/>
+  </inertial>
+  <visual>
+    <origin xyz="-0.04 0.029 -0.44" rpy="0 0 0"/>
+    <geometry>
+      <mesh filename="file://$(find URDF_F_description)/meshes/thighJ_L_1.stl" scale="0.001 0.001 0.001"/>
+    </geometry>
+    <material name="silver"/>
+  </visual>
+  <collision>
+    <origin xyz="-0.04 0.029 -0.44" rpy="0 0 0"/>
+    <geometry>
+      <mesh filename="file://$(find URDF_F_description)/meshes/thighJ_L_1.stl" scale="0.001 0.001 0.001"/>
+    </geometry>
+  </collision>
+</link>
+<link name="AK45-36_tpL_1">
+  <inertial>
+    <origin xyz="-3.642919299551295e-15 -4.371503159459072e-17 -3.3306690738754696e-15" rpy="0 0 0"/>
     <mass value="0.34"/>
     <inertia ixx="0.000099" iyy="0.000132" izz="0.000132" ixy="-0.0" iyz="0.0" ixz="0.0"/>
   </inertial>
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